Commit message: Refactor UR5e Gripper MoveIt Configuration
- Removed the deprecated URDF Xacro file for the UR5e robot.
- Added new configuration files for the UR5e gripper, including initial positions, joint limits, kinematics, and controllers.
- Created launch files for various MoveIt functionalities, including demo, move group, RViz integration, and setup assistant.
- Introduced a new package.xml for the UR5e gripper MoveIt configuration.
- Deleted obsolete test.py file to clean up the repository.

Udapte: New Reference controller
HITL (Moveit RRT* based) updated

File: src/ur5e_gripper_moveit_config/config/ur5e.ros2_control.xacro (robot description, xacro)
@@ -1,5 +1,5 @@
 <?xml version="1.0"?>
 <robot xmlns:xacro="http://www.ros.org/wiki/xacro">
-    <xacro:macro name="ur5e_robot_ros2_control" params="name initial_positions_file">
+    <xacro:macro name="ur5e_ros2_control" params="name initial_positions_file">
         <xacro:property name="initial_positions" value="${load_yaml(initial_positions_file)['initial_positions']}"/>
         <ros2_control name="${name}" type="system">
@@ -11,5 +11,4 @@
                 <command_interface name="position"/>
                 <command_interface name="velocity"/>
-                <command_interface name="effort"/>
                 <state_interface name="position">
                   <param name="initial_value">${initial_positions['shoulder_pan_joint']}</param>
@@ -21,5 +20,4 @@
                 <command_interface name="position"/>
                 <command_interface name="velocity"/>
-                <command_interface name="effort"/>
                 <state_interface name="position">
                   <param name="initial_value">${initial_positions['shoulder_lift_joint']}</param>
@@ -31,5 +29,4 @@
                 <command_interface name="position"/>
                 <command_interface name="velocity"/>
-                <command_interface name="effort"/>
                 <state_interface name="position">
                   <param name="initial_value">${initial_positions['elbow_joint']}</param>
@@ -41,5 +38,4 @@
                 <command_interface name="position"/>
                 <command_interface name="velocity"/>
-                <command_interface name="effort"/>
                 <state_interface name="position">
                   <param name="initial_value">${initial_positions['wrist_1_joint']}</param>
@@ -51,5 +47,4 @@
                 <command_interface name="position"/>
                 <command_interface name="velocity"/>
-                <command_interface name="effort"/>
                 <state_interface name="position">
                   <param name="initial_value">${initial_positions['wrist_2_joint']}</param>
@@ -61,5 +56,4 @@
                 <command_interface name="position"/>
                 <command_interface name="velocity"/>
-                <command_interface name="effort"/>
                 <state_interface name="position">
                   <param name="initial_value">${initial_positions['wrist_3_joint']}</param>
